Commit message: dodanie plików yaml

File: src/hal/urdf/macros.xacro (robot description, xacro)
@@ -64,5 +64,5 @@
   <kp  value="0.0" />
   <kd  value="0.0" />
-  <fdir1 value="1 0 0"/>
+  <!-- <fdir1 value="1 0 0"/> -->
   <material>Gazebo/Red</material>
 </gazebo>
@@ -120,5 +120,5 @@
   <kp  value="0.0" />
   <kd  value="0.0" />
-  <fdir1 value="1 0 0"/>
+  <!-- <fdir1 value="1 0 0"/> -->
   <material>Gazebo/Black</material>
 </gazebo>
@@ -149,14 +149,14 @@
   <inertial>
     <origin xyz="0 0 0" rpy="0 ${PI/2} ${PI/2}" />
-    <mass value="${wheelMass}"/>
+   <mass value="${wheelMass}"/>
     <cylinder_inertia m="${wheelMass}" r="${wheelRadius}" h="${wheelWidth}"/>
-  </inertial>
+</inertial>
 </link>
 <gazebo reference="${lr}_${fmb}_wheel">
-  <mu1 value="1.0"/>
-  <mu2 value="1.0"/>
-  <kp  value="0.0" />
-  <kd  value="0.0" />
-  <fdir1 value="1 0 0"/>
+  <mu1 value="200.0"/>
+  <mu2 value="100.0"/>
+  <kp  value="100000000.0" />
+  <kd  value="1.0" />
+  <!-- <fdir1 value="1 0 0"/> -->
   <material>Gazebo/Black</material>
 </gazebo>
@@ -166,14 +166,16 @@
 <origin xyz="${tX*length_rb*1.41/2} ${tY*width_rb/2+tY*wheelWidth/2} ${tZ*length_rb*1.41/2}" rpy="0 0 0" />
   <axis xyz="0 1 0" rpy="0 0 0" />
-  <limit effort="1" velocity="10"/>
-  <joint_properties damping="0.1" friction="1.0"/>
+  <limit effort="1" velocity="0"/>
+  <joint_properties damping="0.1" friction="0.02"/>
 </joint>
 <transmission name="${lr}_${fmb}_trans">
   <type>transmission_interface/SimpleTransmission</type>
-  <joint name="${lr}_${fmb}_wheel_hinge"/>
   <actuator name="${lr}_${fmb}_Motor">
-    <hardwareInterface>EffortJointInterface</hardwareInterface>
+    <!-- <hardwareInterface>EffortJointInterface</hardwareInterface> -->
     <mechanicalReduction>10</mechanicalReduction>
   </actuator>
+  <joint name="${lr}_${fmb}_wheel_hinge">
+      <hardwareInterface>VelocityJointInterface</hardwareInterface>
+  </joint>
 </transmission>
 </xacro:macro>

File: src/hal/urdf/my1model.xacro (robot description, xacro)
@@ -8,5 +8,5 @@
 <xacro:property name="chassisMass" value="0.2"/>
 <xacro:property name="wheelWidth" value="0.05"/>
-<xacro:property name="wheelRadius" value="0.07"/>
+<xacro:property name="wheelRadius" value="0.04"/>
 <xacro:property name="wheelPos" value="0.2"/>
 <xacro:property name="wheelMass" value="0.3"/>
@@ -49,4 +49,8 @@
   </inertial>
 </link>
+<rocker  lr="left" tY="1"/>
+<rocker  lr="right" tY="-1"/>
+<bogie  lr="left" tY="1"/>
+<bogie  lr="right" tY="-1"/>
 <wheel  lr="left" tY="1" fmb="front" tX="1" rb="bogie" tZ="-1" width_rb="${bogieWidth}" length_rb="${bogieLength}"/>
 <wheel  lr="right" tY="-1" fmb="front" tX="1" rb="bogie" tZ="-1" width_rb="${bogieWidth}" length_rb="${bogieLength}"/>
@@ -55,7 +59,8 @@
 <wheel  lr="left" tY="1" fmb="back" tX="-1" rb="rocker" tZ="-1" width_rb="${rockerWidth}" length_rb="${rockerLengthBack}"/>
 <wheel  lr="right" tY="-1" fmb="back" tX="-1" rb="rocker" tZ="-1" width_rb="${rockerWidth}" length_rb="${rockerLengthBack}"/>
-<rocker  lr="left" tY="1"/>
-<rocker  lr="right" tY="-1"/>
-<bogie  lr="left" tY="1"/>
-<bogie  lr="right" tY="-1"/>
+<gazebo>
+  <plugin name="gazebo_ros_control" filename="libgazebo_ros_control.so">
+    <robotNamespace>/</robotNamespace>
+  </plugin>
+</gazebo>
 </robot>

Commit message: Rviz, gazebo, imu, ekf_nodes

File: src/hal/urdf/macros.xacro (robot description, xacro)
@@ -20,4 +20,186 @@
   />
 </xacro:macro>
+<xacro:macro name="camera">
+<!-- Camera -->
+  <link name="camera_link">
+    <collision>
+      <origin xyz="0 0 0" rpy="0 0 0"/>
+      <geometry>
+    <box size="${cameraSize} ${cameraSize} ${cameraSize}"/>
+      </geometry>
+    </collision>
+    <visual>
+      <origin xyz="0 0 0" rpy="0 0 0"/>
+      <geometry>
+        <box size="${cameraSize} ${cameraSize} ${cameraSize}"/>
+      </geometry>
+    </visual>
+    <inertial>
+      <mass value="${cameraMass}" />
+      <origin xyz="0 0 0" rpy="0 0 0"/>
+        <box_inertia m="${cameraMass}" x="${cameraSize}" y="${cameraSize}" z="${cameraSize}"/>
+    </inertial>
+  </link>
+<joint name="camera_joint" type="fixed">
+    <axis xyz="0 1 0" />
+    <origin xyz="${chassisLength/2 - cameraSize/2} 0 ${chassisHeight/2 + cameraSize/2}" rpy="0 0 0"/>
+    <parent link="base_link"/>
+    <child link="camera_link"/>
+  </joint>
+<gazebo reference="camera_link">
+      <material>Gazebo/Red</material>
+    <sensor type="camera" name="camera1">
+      <update_rate>30.0</update_rate>
+      <plugin name="camera_controller" filename="libgazebo_ros_camera.so">
+      <!-- <horizontal_fov>0.5</horizontal_fov>
+        <image>
+          <width>1960</width>
+          <height>1080</height>
+          <format>R8G8B8</format>
+        </image>
+        <clip>
+          <near>0.02</near>
+          <far>300</far>
+        </clip> -->
+        <!-- <noise>
+          <type>gaussian</type>
+          Noise is sampled independently per pixel on each frame.
+               That pixel's noise value is added to each of its color
+               channels, which at that point lie in the range [0,1].
+          <mean>0.0</mean>
+          <stddev>0.007</stddev>
+        </noise> -->
+        <alwaysOn>true</alwaysOn>
+        <updateRate>0.0</updateRate>
+        <cameraName>camera1</cameraName>
+        <imageTopicName>image_raw</imageTopicName>
+        <cameraInfoTopicName>camera_info</cameraInfoTopicName>
+        <frameName>camera_link</frameName>
+        <hackBaseline>0.07</hackBaseline>
+        <distortionK1>0.0</distortionK1>
+        <distortionK2>0.0</distortionK2>
+        <distortionK3>0.0</distortionK3>
+        <distortionT1>0.0</distortionT1>
+        <distortionT2>0.0</distortionT2>
+      </plugin>
+      <image>
+          <width>1960</width>
+          <height>1080</height>
+          <format>R8G8B8</format>
+        </image>
+    </sensor>
+  </gazebo>
+</xacro:macro>
+<xacro:macro name="imu">
+<link name="imu">
+<collision>
+  <origin xyz="0 0 0" rpy="0 0 0" />
+    <geometry>
+      <box size="${imuSize} ${imuSize} ${imuSize}"/>
+    </geometry>
+</collision>
+  <visual>
+  <origin xyz="0 0 0" rpy="0 0 0" />
+    <geometry>
+            <box size="${imuSize} ${imuSize} ${imuSize}"/>
+    </geometry>
+  </visual>
+  <inertial>
+  <origin xyz="0 0 0" rpy="0 0 0" />
+      <mass value="${imuMass}"/>
+      <box_inertia m="${imuMass}" x="${imuSize}" y="${imuSize}" z="${imuSize}"/>
+  </inertial>
+</link>
+<joint name="imu_joint" type="fixed">
+  <parent link="base_link"/>
+  <child link="imu"/>
+  <origin xyz="0 0 ${chassisHeight/2 + imuSize/2}" rpy="0 0 0" />
+</joint>
+  <gazebo reference="imu">
+    <material>Gazebo/Red</material>
+    <gravity>true</gravity>
+    <sensor type="imu" name="imu_sensor1" >
+      <always_on>true</always_on>
+      <update_rate>100</update_rate>
+      <visualize>true</visualize>
+      <topic>__default_topic__</topic>
+      <plugin filename="libgazebo_ros_imu_sensor.so" name="imu_plugin">
+        <topicName>imu/data</topicName>
+        <bodyName>imu_link</bodyName>
+        <updateRateHZ>10.0</updateRateHZ>
+        <gaussianNoise>0.0</gaussianNoise>
+        <xyzOffset>0 0 0</xyzOffset>
+        <rpyOffset>0 0 0</rpyOffset>
+        <frameName>imu</frameName>
+      </plugin>
+      <pose>0 0 0 0 0 0</pose>
+    </sensor>
+  </gazebo>
+</xacro:macro>
+<xacro:macro name="lidar">
+<link name="lidar">
+<collision>
+  <origin xyz="0 0 0" rpy="0 0 0" />
+    <geometry>
+      <box size="${lidarSize} ${lidarSize} ${lidarSize}"/>
+    </geometry>
+</collision>
+  <visual>
+  <origin xyz="0 0 0" rpy="0 0 0" />
+    <geometry>
+      <mesh filename="model://hokuyo/meshes/hokuyo.dae"/>
+    </geometry>
+  </visual>
+  <inertial>
+  <origin xyz="0 0 0" rpy="0 0 0" />
+      <mass value="${lidarMass}"/>
+      <box_inertia m="${lidarMass}" x="${lidarSize}" y="${lidarSize}" z="${lidarSize}"/>
+  </inertial>
+</link>
+<gazebo reference="lidar">
+  <mu1 value="100.0"/>
+  <mu2 value="100.0"/>
+  <kp  value="10000.0" />
+  <kd  value="1.0" />
+  <sensor type="ray" name="head_hokuyo_sensor">
+      <pose>0 0 0 0 0 0</pose>
+      <visualize>true</visualize>
+      <update_rate>40</update_rate>
+      <ray>
+        <scan>
+          <horizontal>
+            <samples>720</samples>
+            <resolution>1</resolution>
+            <min_angle>-2.09</min_angle>
+            <max_angle>2.09</max_angle>
+          </horizontal>
+        </scan>
+        <range>
+          <min>0.10</min>
+          <max>3.0</max>
+          <resolution>0.01</resolution>
+        </range>
+        <noise>
+          <type>gaussian</type>
+          <!-- Noise parameters based on published spec for Hokuyo laser
+               achieving "+-30mm" accuracy at range < 10m.  A mean of 0.0m and
+               stddev of 0.01m will put 99.7% of samples within 0.03m of the true
+               reading. -->
+          <mean>0.0</mean>
+          <stddev>0.01</stddev>
+        </noise>
+      </ray>
+      <plugin name="gazebo_ros_head_hokuyo_controller" filename="libgazebo_ros_laser.so">
+        <topicName>lidar/scan</topicName>
+        <frameName>lidar</frameName>
+      </plugin>
+    </sensor>
+</gazebo>
+<joint name="lidar" type="fixed">
+  <parent link="base_link"/>
+  <child link="lidar"/>
+  <origin xyz="${chassisLength/2 - lidarSize/2} 0 ${-chassisHeight/2 - lidarSize/2}" rpy="${PI} 0 0" />
+</joint>
+</xacro:macro>
 <xacro:macro name ="rocker" params="lr tY">
 <link name="${lr}_rocker">
@@ -33,5 +215,4 @@
        <box size="${rockerLengthFront} ${rockerWidth} ${rockerWidth}"/>
     </geometry>
-    <material name="blue"/>
   </visual>
   <inertial>
@@ -51,5 +232,4 @@
        <box size="${rockerLengthBack} ${rockerWidth} ${rockerWidth}"/>
     </geometry>
-    <material name="black"/>
   </visual>
   <inertial>
@@ -60,18 +240,17 @@
 </link>
 <gazebo reference="${lr}_rocker">
-  <mu1 value="1.0"/>
-  <mu2 value="1.0"/>
-  <kp  value="0.0" />
-  <kd  value="0.0" />
-  <!-- <fdir1 value="1 0 0"/> -->
+  <mu1 value="100.0"/>
+  <mu2 value="100.0"/>
+  <kp  value="10000.0" />
+  <kd  value="1.0" />
   <material>Gazebo/Red</material>
 </gazebo>
-<joint name="${lr}_rocker_hinge" type="revolute">
-  <parent link="chassis"/>
+<joint name="${lr}_rocker_hinge" type="fixed">
+  <parent link="base_link"/>
   <child link="${lr}_rocker"/>
   <origin xyz="0 ${tY*rockerWidth/2+tY*chassisWidth/2} 0" rpy="0 0 0" />
-  <axis xyz="0 1 0" rpy="0 0 0" />
-  <limit effort="1" lower="${-PI/6}" upper="${PI/6}" velocity="0.0001"/>
-  <joint_properties damping="0.0" friction="0.0"/>
+  <!-- <axis xyz="0 1 0" rpy="0 0 0" />
+  <limit effort="100" lower="${-PI/24}" upper="${PI/24}" velocity="0.0001"/>
+  <joint_properties damping="0.2" friction="0.6"/> -->
 </joint>
 </xacro:macro>
@@ -89,5 +268,4 @@
        <box size="${bogieLength} ${bogieWidth} ${bogieWidth}"/>
     </geometry>
-    <material name="blue"/>
   </visual>
   <inertial>
@@ -107,5 +285,4 @@
        <box size="${bogieLength} ${bogieWidth} ${bogieWidth}"/>
     </geometry>
-    <material name="blue"/>
   </visual>
   <inertial>
@@ -116,9 +293,8 @@
 </link>
 <gazebo reference="${lr}_bogie">
-  <mu1 value="1.0"/>
-  <mu2 value="1.0"/>
-  <kp  value="0.0" />
-  <kd  value="0.0" />
-  <!-- <fdir1 value="1 0 0"/> -->
+  <mu1 value="100.0"/>
+  <mu2 value="100.0"/>
+  <kp  value="10000.0" />
+  <kd  value="1.0" />
   <material>Gazebo/Black</material>
 </gazebo>
@@ -128,6 +304,6 @@
 <origin xyz="${rockerLengthFront*1.41/2} ${tY*rockerWidth/2+tY*bogieWidth/2} -${rockerLengthFront*1.41/2}" rpy="0 0 0" />
   <axis xyz="0 1 0" rpy="0 0 0" />
-  <limit effort="1" lower="${-PI/6}" upper="${PI/6}" velocity="0.0001"/>
-  <joint_properties damping="0.0" friction="0.0"/>
+  <limit effort="100" lower="${-PI/6}" upper="${PI/6}" velocity="0.0001"/>
+  <joint_properties damping="0.0  " friction="0.0"/>
 </joint>
 </xacro:macro>
@@ -154,28 +330,38 @@
 </link>
 <gazebo reference="${lr}_${fmb}_wheel">
-  <mu1 value="200.0"/>
+  <mu1 value="100.0"/>
   <mu2 value="100.0"/>
-  <kp  value="100000000.0" />
+  <kp  value="100000.0" />
   <kd  value="1.0" />
-  <!-- <fdir1 value="1 0 0"/> -->
   <material>Gazebo/Black</material>
 </gazebo>
 <joint name="${lr}_${fmb}_wheel_hinge" type="continuous">
+  <axis xyz="0 1 0" rpy="0 0 0" />
   <parent link="${lr}_${rb}"/>
   <child link="${lr}_${fmb}_wheel"/>
-<origin xyz="${tX*length_rb*1.41/2} ${tY*width_rb/2+tY*wheelWidth/2} ${tZ*length_rb*1.41/2}" rpy="0 0 0" />
-  <axis xyz="0 1 0" rpy="0 0 0" />
-  <limit effort="1" velocity="0"/>
-  <joint_properties damping="0.1" friction="0.02"/>
-</joint>
-<transmission name="${lr}_${fmb}_trans">
+  <origin xyz="${tX*length_rb*1.41/2} ${tY*width_rb/2+tY*wheelWidth/2} ${tZ*length_rb*1.41/2}" rpy="0 0 0" />
+  <!-- <limit effort="1" velocity="0"/>
+  <joint_properties damping="0.1" friction="0.02"/> -->
+</joint>
+<!-- <transmission name="${lr}_${fmb}_trans">
   <type>transmission_interface/SimpleTransmission</type>
   <actuator name="${lr}_${fmb}_Motor">
-    <!-- <hardwareInterface>EffortJointInterface</hardwareInterface> -->
+    <hardwareInterface>EffortJointInterface</hardwareInterface>
     <mechanicalReduction>10</mechanicalReduction>
   </actuator>
   <joint name="${lr}_${fmb}_wheel_hinge">
-      <hardwareInterface>VelocityJointInterface</hardwareInterface>
+      <hardwareInterface>hardware_interface/VelocityJointInterface</hardwareInterface>
+  </joint>z
+</transmission>
+-->
+<transmission name="${lr}_${fmb}_trans">
+  <type>transmission_interface/SimpleTransmission</type>
+  <joint name="${lr}_${fmb}_wheel_hinge">
+      <hardwareInterface>hardware_interface/VelocityJointInterface</hardwareInterface>
   </joint>
+  <actuator name="${lr}_${fmb}_Motor">
+      <hardwareInterface>hardware_interface/VelocityJointInterface</hardwareInterface>
+      <mechanicalReduction>1</mechanicalReduction>
+  </actuator>
 </transmission>
 </xacro:macro>

Commit message: konfiguracja

File: src/hal/urdf/macros.xacro (robot description, xacro)
@@ -137,4 +137,43 @@
   </gazebo>
 </xacro:macro>
+<xacro:macro name="gps">
+<link name="gps">
+<collision>
+  <origin xyz="0 0 0" rpy="0 0 0" />
+    <geometry>
+      <box size="${gpsSize} ${gpsSize} ${gpsSize}"/>
+    </geometry>
+</collision>
+  <visual>
+  <origin xyz="0 0 0" rpy="0 0 0" />
+    <geometry>
+            <box size="${gpsSize} ${gpsSize} ${gpsSize}"/>
+    </geometry>
+  </visual>
+  <inertial>
+  <origin xyz="0 0 0" rpy="0 0 0" />
+      <mass value="${gpsMass}"/>
+      <box_inertia m="${gpsMass}" x="${gpsSize}" y="${gpsSize}" z="${gpsSize}"/>
+  </inertial>
+</link>
+<joint name="gps_joint" type="fixed">
+  <parent link="base_link"/>
+  <child link="gps"/>
+  <origin xyz="0 0 ${-chassisHeight/2 - gpsSize/2}" rpy="0 0 0" />
+</joint>
+<gazebo>
+    <plugin name="novatel_gps_sim" filename="libhector_gazebo_ros_gps.so">
+      <alwaysOn>1</alwaysOn>
+      <updateRate>10.0</updateRate>
+      <bodyName>base_link</bodyName>
+      <topicName>gps/fix</topicName>
+      <velocityTopicName>gps/fix_velocity</velocityTopicName>
+      <drift>5.0 5.0 5.0</drift>
+      <gaussianNoise>0.1 0.1 0.1</gaussianNoise>
+      <velocityDrift>0 0 0</velocityDrift>
+      <velocityGaussianNoise>0.1 0.1 0.1</velocityGaussianNoise>
+    </plugin>
+  </gazebo>
+</xacro:macro>
 <xacro:macro name="lidar">
 <link name="lidar">
@@ -191,5 +230,5 @@
       </ray>
       <plugin name="gazebo_ros_head_hokuyo_controller" filename="libgazebo_ros_laser.so">
-        <topicName>lidar/scan</topicName>
+        <topicName>scan</topicName>
         <frameName>lidar</frameName>
       </plugin>
@@ -199,5 +238,6 @@
   <parent link="base_link"/>
   <child link="lidar"/>
-  <origin xyz="${chassisLength/2 - lidarSize/2} 0 ${-chassisHeight/2 - lidarSize/2}" rpy="${PI} 0 0" />
+  <!-- <origin xyz="${chassisLength/2 - lidarSize/2} 0 ${-chassisHeight/2 - lidarSize/2}" rpy="${PI} 0 0" /> -->
+    <origin xyz="${chassisLength/2 - lidarSize/2} 0 ${chassisHeight/2 +cameraSize + lidarSize/2+0.01}" rpy="0 0 0" />
 </joint>
 </xacro:macro>
@@ -341,18 +381,5 @@
   <child link="${lr}_${fmb}_wheel"/>
   <origin xyz="${tX*length_rb*1.41/2} ${tY*width_rb/2+tY*wheelWidth/2} ${tZ*length_rb*1.41/2}" rpy="0 0 0" />
-  <!-- <limit effort="1" velocity="0"/>
-  <joint_properties damping="0.1" friction="0.02"/> -->
-</joint>
-<!-- <transmission name="${lr}_${fmb}_trans">
-  <type>transmission_interface/SimpleTransmission</type>
-  <actuator name="${lr}_${fmb}_Motor">
-    <hardwareInterface>EffortJointInterface</hardwareInterface>
-    <mechanicalReduction>10</mechanicalReduction>
-  </actuator>
-  <joint name="${lr}_${fmb}_wheel_hinge">
-      <hardwareInterface>hardware_interface/VelocityJointInterface</hardwareInterface>
-  </joint>z
-</transmission>
--->
+</joint>
 <transmission name="${lr}_${fmb}_trans">
   <type>transmission_interface/SimpleTransmission</type>
@@ -366,3 +393,77 @@
 </transmission>
 </xacro:macro>
+<xacro:macro name="wheel2" params="lr tY fmb tX rb tZ width_rb length_rb">
+<link name="${lr}_${fmb}_wheel">
+  <collision>
+    <origin xyz="0 0 0" rpy="0 ${PI/2} ${PI/2}" />
+    <geometry>
+      <cylinder length="${wheelWidth}" radius="${wheelRadius}"/>
+    </geometry>
+  </collision>
+  <visual>
+    <origin xyz="0 0 0" rpy="0 ${PI/2} ${PI/2}" />
+    <geometry>
+      <cylinder length="${wheelWidth}" radius="${wheelRadius}"/>
+    </geometry>
+    <material name="black"/>
+  </visual>
+  <inertial>
+    <origin xyz="0 0 0" rpy="0 ${PI/2} ${PI/2}" />
+   <mass value="${wheelMass}"/>
+    <cylinder_inertia m="${wheelMass}" r="${wheelRadius}" h="${wheelWidth}"/>
+</inertial>
+</link>
+<gazebo reference="${lr}_${fmb}_wheel">
+  <mu1 value="100.0"/>
+  <mu2 value="100.0"/>
+  <kp  value="100000.0" />
+  <kd  value="1.0" />
+  <material>Gazebo/Black</material>
+</gazebo>
+<joint name="${lr}_${fmb}_wheel_hinge" type="continuous">
+  <axis xyz="0 1 0" rpy="0 0 0" />
+  <parent link="base_link"/>
+  <child link="${lr}_${fmb}_wheel"/>
+  <origin xyz="0 ${tY*chassisWidth/2+tY*wheelWidth/2} 0" rpy="0 0 0" />
+</joint>
+<transmission name="${lr}_${fmb}_trans">
+  <type>transmission_interface/SimpleTransmission</type>
+  <joint name="${lr}_${fmb}_wheel_hinge">
+      <hardwareInterface>hardware_interface/VelocityJointInterface</hardwareInterface>
+  </joint>
+  <actuator name="${lr}_${fmb}_Motor">
+      <hardwareInterface>hardware_interface/VelocityJointInterface</hardwareInterface>
+      <mechanicalReduction>1</mechanicalReduction>
+  </actuator>
+</transmission>
+</xacro:macro>
+  <xacro:macro name="sphere_inertia" params="m r">
+    <inertial>
+      <mass value="${m}"/>
+      <inertia ixx="${2.0*m*(r*r)/5.0}" ixy="0.0" ixz="0.0" iyy="${2.0*m*(r*r)/5.0}" iyz="0.0" izz="${2.0*m*(r*r)/5.0}"/>
+    </inertial>
+  </xacro:macro>
+ <xacro:macro name="caster" params="fb tX">
+   <link name="${fb}_caster_wheel">
+    <visual>
+      <origin xyz="0 0 0" rpy="0 0 0"/>
+      <geometry>
+        <sphere radius="${caster_wheel_radius}"/>
+      </geometry>
+    </visual>
+    <collision>
+      <origin xyz="0 0 0" rpy="0 0 0"/>
+      <geometry>
+        <sphere radius="${caster_wheel_radius}"/>
+      </geometry>
+    </collision>
+    <xacro:sphere_inertia m="5" r="${caster_wheel_radius}"/>
+  </link>
+  <joint name="${fb}_caster_wheel_joint" type="continuous">
+    <axis xyz="0 1 0" rpy="0 0 0" />
+    <parent link="base_link"/>
+    <child link="${fb}_caster_wheel"/>
+    <origin xyz="${tX*chassisLength/2-tX*caster_wheel_radius} 0 ${-chassisHeight/2}" rpy="0 0 0"/>
+  </joint>
+</xacro:macro>
 </robot>

File: src/hal/urdf/my1model.urdf (robot description, URDF)
Before this commit: robot my1model, 2 links, 1 joints
Joints:
- joint base_joint: origin xyz=0 0 ${wheelRadius+rockerLengthBack*1.41/2} rpy=0 0 0 -> xyz=0 0 ${wheelRadius} rpy=0 0 0

Commit message: 200lat póżniej....DZIAŁA!

File: src/hal/urdf/macros.xacro (robot description, xacro)
@@ -50,5 +50,5 @@
       <material>Gazebo/Red</material>
     <sensor type="camera" name="camera1">
-      <update_rate>30.0</update_rate>
+      <update_rate>10.0</update_rate>
       <plugin name="camera_controller" filename="libgazebo_ros_camera.so">
       <!-- <horizontal_fov>0.5</horizontal_fov>
@@ -137,6 +137,6 @@
   </gazebo>
 </xacro:macro>
-<xacro:macro name="gps">
-<link name="gps">
+<xacro:macro name="gps" params="freq color name shift drift noise vel_drift vel_noise">
+<link name="gps_${name}">
 <collision>
   <origin xyz="0 0 0" rpy="0 0 0" />
@@ -157,21 +157,27 @@
   </inertial>
 </link>
-<joint name="gps_joint" type="fixed">
+<joint name="gps_joint_${name}" type="fixed">
   <parent link="base_link"/>
-  <child link="gps"/>
-  <origin xyz="0 0 ${-chassisHeight/2 - gpsSize/2}" rpy="0 0 0" />
+  <child link="gps_${name}"/>
+  <origin xyz="0 0 ${-chassisHeight/2 - gpsSize/2-shift}" rpy="0 0 0" />
 </joint>
 <gazebo>
-    <plugin name="novatel_gps_sim" filename="libhector_gazebo_ros_gps.so">
-      <alwaysOn>1</alwaysOn>
-      <updateRate>10.0</updateRate>
-      <bodyName>base_link</bodyName>
-      <topicName>gps/fix</topicName>
-      <velocityTopicName>gps/fix_velocity</velocityTopicName>
-      <drift>5.0 5.0 5.0</drift>
-      <gaussianNoise>0.1 0.1 0.1</gaussianNoise>
-      <velocityDrift>0 0 0</velocityDrift>
-      <velocityGaussianNoise>0.1 0.1 0.1</velocityGaussianNoise>
-    </plugin>
+  <material>Gazebo/${color}</material>
+  <plugin name="gps_controller" filename="libhector_gazebo_ros_gps.so">
+    <alwaysOn>true</alwaysOn>
+    <updateRate>${freq}</updateRate>
+    <robotNamespace>${name}</robotNamespace>
+    <bodyName>gps_${name}</bodyName>
+    <frameId>map</frameId>
+    <!-- <topicname>/gps/fix</topicname>
+    <velocitytopicname>/gps/fix_velocity</velocitytopicname> -->
+    <!-- <drift>5.0 5.0 5.0</drift> -->
+    <drift>${drift} ${drift} ${drift}</drift>
+    <gaussianNoise>${noise} ${noise} ${noise}</gaussianNoise>
+    <!-- <driftFrequency>${noise} ${noise} ${noise}</driftFrequency> -->
+    <velocityDrift>${vel_drift} ${vel_drift} ${vel_drift}</velocityDrift>
+    <velocityGaussianNoise>${vel_noise} ${vel_noise} ${vel_noise}</velocityGaussianNoise>
+    <!-- <velocitygaussiannoise>0.1 0.1 0.1</velocitygaussiannoise> -->
+</plugin>
   </gazebo>
 </xacro:macro>

File: src/hal/urdf/my1model.urdf (robot description, URDF)
Before this commit: robot my1model, 2 links, 1 joints
Joints:
- joint base_joint: origin xyz=0 0 ${wheelRadius} rpy=0 0 0 -> xyz=0 0 ${wheelRadius+rockerLengthBack*1.41/2} rpy=0 0 0
